Commit message: vinger-GLB's hergecalibreerd (dichtstand) + Hand-E in de foxglove-URDF

File: ur5e_hand_e/ur5e_hand_e_foxglove.urdf (robot description, URDF)
Before this commit: robot ur5e, 11 links, 10 joints
Links:
- added link hand_e; visual mesh filename=../cel/hand_e.glb
- added link vinger_min; visual mesh filename=../cel/hand_e_vinger_min.glb
- added link vinger_plus; visual mesh filename=../cel/hand_e_vinger_plus.glb
Joints:
- added joint Slider_1: type prismatic, parent tool0, child vinger_min, origin xyz=0 0 0 rpy=0 0 0, axis -1 0 0, limit lower=0.0 upper=0.025 effort=60.0 velocity=0.15
- added joint Slider_2: type prismatic, parent tool0, child vinger_plus, origin xyz=0 0 0 rpy=0 0 0, axis 1 0 0, limit lower=0.0 upper=0.025 effort=60.0 velocity=0.15
- added joint tool0-hand_e: type fixed, parent tool0, child hand_e, origin xyz=0 0 0 rpy=0 0 0

Commit message: Hand-E-behuizing zwart (materiaalloos stage-artefact) + ?v=7 op de hand-meshes

File: ur5e_hand_e/ur5e_hand_e_foxglove.urdf (robot description, URDF)
Before this commit: robot ur5e, 14 links, 13 joints
Links:
- link hand_e: geometry visual mesh filename=../cel/hand_e.glb?v=7
- link vinger_min: geometry visual mesh filename=../cel/hand_e_vinger_min.glb?v=7
- link vinger_plus: geometry visual mesh filename=../cel/hand_e_vinger_plus.glb?v=7
